File: board/FrontPanel.sch (EAGLE design)
At the start: 0 parts

Commit message: Front panel design with dimension markings
Parts:
- added J1: PINHD-1X2BIG, SaintGimp:PINHD-1X2BIG
- added S1, S2, S3, S4: SWITCH-MOMENTARY-6MM, SaintGimp:SWITCH-MOMENTARY-6MM
Connections:
- new net N$1: J11.KL, S1.1, S1.2, S2.1, S2.2, S3.1, S3.2, S4.1, S4.2
- new net N$2: J12.KL, S1.3, S1.4, S2.3, S2.4, S3.3, S3.4, S4.3, S4.4
